File: KiCAD project/kicad_project_geiger.kicad_pcb (KiCad board)
At the start: 2 copper layers, 66.8 x 104.8 mm, 66 parts, among them P4 I ROVER, P7 BATTERY, Q1 2SC1815, Q2 2SC1815, SW1 SWITCH_INV, SW2 SW_DIP_3, SW4 2MD3T2B2M2RE, U1 FGPMMOPA6H, U10 MIC5205, U11 piezo_buzzer, U12 stereo_audio_socket, U2 MAX1555, U3 XBee, U4 OLED-PCB, U5 SD_CARD_SLOT, U6 MCP1826S, U7 RedBear, U8 LSM303C, U9 LM3880

Commit message: Update
Parts:
- removed C16: 100nF, RedBear:R_0603_HandSoldering
- removed G***: LOGO, OPENHARDWARE:OSHWLOGO1.5IN
- removed U12: stereo_audio_socket, CLIFF_ELECTRONIC_COMPONENTS_FC68131_PhoneAudioConnector:CLIFF_ELECTRONIC_COMPONENTS_FC68131_PhoneAudioConnector
- added L1: Ferrite, RedBear:R_0603_HandSoldering, F.Cu at (134.5, 98.1)
- added P1: uFL_conn, UFL-R-SMT:U.FL-R-SMT, F.Cu at (116.4, 116.1)
- added Q3: RSR010N10FHATL, sot_32_standard:SOT-23, F.Cu at (46.3, 192.8)
- added Q4: ZXMP6A13F, sot_32_standard:SOT-23, F.Cu at (33.0, 183.5)
- added Q5: BC847C, sot_32_standard:SOT-23, B.Cu at (166.0, 65.2)
- added Q6: RSR010N10FHATL, sot_32_standard:SOT-23, B.Cu at (144.1, 54.2)
- added Q7: RSR010N10FHATL, sot_32_standard:SOT-23, F.Cu at (134.0, 69.5)
- added R20: 68R, RedBear:R_0603_HandSoldering, B.Cu at (152.5, 57.7)
- added R21: 10K, RedBear:R_0603_HandSoldering, F.Cu at (141.8, 69.6)
- added R22: 10K, RedBear:R_0603_HandSoldering, F.Cu at (139.4, 69.6)
- added R23: 10K, RedBear:R_0603_HandSoldering, F.Cu at (137.2, 69.6)
- added R24: 0K, RedBear:R_0603_HandSoldering, B.Cu at (144.6, 57.7)
- added R25: 0K, RedBear:R_0603_HandSoldering, B.Cu at (139.8, 57.7)
- added SW3: SWITCH_INV, OS102011MA1QN1_slide_switch:OS102011MA1QN1_slide_switch, F.Cu at (173.0, 84.6)
- C13, C14, C15, R11, R13, R4, R5, R9, U2: moved to B.Cu
- D2: footprint RedBear:LED_0603_HandSoldering -> KPD-3224SURCK:KPD-3224SURCK
- D3: value BLUE -> GREEN; footprint LEDs:LED-5MM -> MCL053SGC:MCL053SGC
- D4: footprint RedBear:1N4148 -> SOD-323_standard:SOD-323; moved to B.Cu
- D6: value 1N4148 -> BAT20J; footprint RedBear:1N4148 -> SOD-323_standard:SOD-323; moved to B.Cu
- P4: footprint Socket_Strips:Socket_Strip_Angled_1x03 -> B3B-PH-SM4-TB_IROVER_CONNECTOR:B3B-PH-SM4-TB_IROVER_CONNECTOR
- Q1: value 2SC1815 -> ZXMP6A13F; footprint 2SC1815:TO-92_Inline_Narrow_Oval -> sot_32_standard:SOT-23; moved to B.Cu
- Q2: value 2SC1815 -> RSR010N10FHATL; footprint 2SC1815:TO-92_Inline_Narrow_Oval -> sot_32_standard:SOT-23; moved to B.Cu
- R12: value 1K -> 10K; moved to B.Cu
- R14: value 100K -> 51K; moved to B.Cu
- R15: value 47K -> 10K
- R16: value 4.7K -> 10K
- R19: value 180K -> 10K
- R8: value 10K -> 100K; moved to B.Cu
- SW4: value 2MD3T2B2M2RE -> SW_PUSH; footprint TSM102C3_toggle_switch_tme:TSM102C3_toggle_switch -> KSEK43J_LFS_TACTILE_SWITCH:KSEK43J_LFS_TACTILE_SWITCH
- U11: value piezo_buzzer -> buzzer; footprint CEM-1203(42)_piezo_buzzer:CEM-1203(42) -> LD-BZEG-1205:LD-BZEG-1205
- U7: footprint RedBear -> RedBear:RedBear
- moved R16 168.9 mm to (17.4, 192.7), turned to 0 degrees
- moved R15 157.6 mm to (26.0, 188.2), turned to 0 degrees
- moved C5 116.3 mm to (132.1, 188.7), turned to 0 degrees
- moved C2 114.4 mm to (99.2, 174.4), turned to 0 degrees
- moved U6 106.1 mm to (119.4, 181.7), turned to 0 degrees
- moved C10 95.5 mm to (146.3, 175.4), turned to 0 degrees
- moved D6 79.3 mm to (158.2, 137.0), turned to 270 degrees
- moved R17 78.1 mm to (54.5, 166.1), turned to 270 degrees
- moved D1 75.6 mm to (58.5, 170.9), turned to 0 degrees
- moved U2 72.1 mm to (158.3, 150.8), turned to 180 degrees
- moved C14 67.1 mm to (151.0, 148.0), turned to 180 degrees
- moved C13 66.6 mm to (151.0, 152.3), turned to 180 degrees
- moved Q1 65.2 mm to (161.9, 136.9), turned to 90 degrees
- moved C1 57.6 mm to (176.4, 121.2)
- moved U3 56.5 mm to (170.7, 121.2), turned to 270 degrees
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Connections:
- C2 pad 1: VBAT -> LDO
- C3 pad 2: +3V3 -> Net-(C3-Pad2)
- D2 pad 1: GND -> Net-(D2-Pad1)
- D6 pad 1: +3V3 -> PWR
- D6 pad 2: Net-(D6-Pad2) -> VUSB
- P7 pad 1: Net-(P7-Pad1) -> VBAT
- Q1 pad 1: GND -> VUSB
- Q1 pad 2: Net-(D3-Pad1) -> PWR
- Q1 pad 3: Net-(Q1-Pad3) -> VBAT
- Q2 pad 1: GND -> AUDIO
- Q2 pad 2: Net-(D6-Pad2) -> GND
- R10 pad 1: Net-(R10-Pad1) -> BAT_MEASURE
- R11 pad 1: Net-(D3-Pad2) -> CNT_LED
- R11 pad 2: Net-(R11-Pad2) -> Net-(D3-Pad2)
- R12 pad 1: Net-(D2-Pad2) -> GND
- R12 pad 2: Net-(R12-Pad2) -> AUDIO
- R14 pad 1: Net-(Q1-Pad3) -> Net-(Q5-Pad1)
- R15 pad 1: Net-(C16-Pad1) -> GND
- R15 pad 2: Net-(R15-Pad2) -> PWR_ON
- R16 pad 1: Net-(R15-Pad2) -> Net-(Q3-Pad3)
- R16 pad 2: GND -> PWR
- R18 pad 1: Net-(D5-Pad2) -> Net-(R18-Pad1)
- R18 pad 2: Net-(R18-Pad2) -> Net-(D5-Pad2)
- R19 pad 1: Net-(R19-Pad1) -> GND
- R19 pad 2: Net-(Q2-Pad3) -> PWR_OFF
- R8 pad 1: +3V3 -> VUSB
- R8 pad 2: LOG_CNT_SEL -> GND
- R9 pad 2: Net-(R10-Pad1) -> BAT_MEASURE
- SW1 pad 1: (no net) -> PWR_OFF
- SW1 pad 2: VBAT -> PWR
- SW1 pad 3: Net-(P7-Pad1) -> LDO
- SW2 pad 2: LOG_ALARM -> +3V3
- SW2 pad 3: IROVER -> +3V3
- SW2 pad 4: Net-(R19-Pad1) -> PIEZO
- SW2 pad 5: Net-(R12-Pad2) -> CNT_LED
- SW2 pad 6: Net-(R11-Pad2) -> LOG_LED
- SW4 pad 1: (no net) -> GND
- SW4 pad 2: LOG_CNT_SEL -> ANALOG
- U1 pad 1: +3V3 -> Net-(C3-Pad2)
- U1 pad 11: (no net) -> Net-(P1-Pad1)
- U1 pad 4: (no net) -> VBAT
- U1 pad 5: Net-(R18-Pad2) -> Net-(R18-Pad1)
- U11 pad 1: +3V3 -> PIEZO
- U11 pad 2: Net-(D6-Pad2) -> Net-(Q2-Pad3)
- U4 pad 1: SPI_MOSI -> I2C_SDA
- U4 pad 2: SPI_SCK -> I2C_SCL
- U4 pad 3: LCD_DC -> Net-(R24-Pad2)
- U4 pad 5: LCD_CS -> GND
- U6 pad 1: VBAT -> LDO
- U7 pad 15: LOG_ALARM -> IROVER
- U7 pad 16: IROVER -> PWR_ON
- U7 pad 17: CS_LOG -> BAT_MEASURE
- U7 pad 18: LOG_CNT_SEL -> ANALOG
- U7 pad 19: Net-(R10-Pad1) -> AUDIO
- U7 pad 20: CD_LOG -> (no net)
- U7 pad 6: LCD_CS -> CS_LOG
- U7 pad 7: LCD_RST -> CD_LOG
- U7 pad 8: LCD_DC -> LCD_RST
Routing:
- net GND: track 494.6 -> 0.00 mm, vias 17 -> 0
- net +3V3: track 338.9 -> 0.00 mm, vias 15 -> 0
- net VBAT: track 239.0 -> 0.00 mm, vias 13 -> 0
- net IROVER: track 148.4 -> 0.00 mm, vias 4 -> 0
- net SPI_SCK: track 141.3 -> 0.00 mm, vias 3 -> 0
- net SPI_MOSI: track 135.8 -> 0.00 mm, vias 3 -> 0
- net LCD_DC: track 103.5 -> 0.00 mm, vias 3 -> 0
- net LCD_CS: track 96.1 -> 0.00 mm, vias 2 -> 0
- net LCD_RST: track 95.1 -> 0.00 mm, vias 2 -> 0
- net VUSB: track 90.2 -> 0.00 mm, vias 2 -> 0
- net Net-(P7-Pad1): track 89.8 -> 0.00 mm
- net Net-(R17-Pad2): track 76.5 -> 0.00 mm, vias 2 -> 0
- net TX_XBEE: track 74.3 -> 0.00 mm, vias 2 -> 0
- net RX_XBEE: track 72.6 -> 0.00 mm, vias 2 -> 0
- net I2C_SDA: track 70.9 -> 0.00 mm, vias 1 -> 0
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- removed copper zone on B.Cu, net GND
- removed copper zone on F.Cu, net GND
Other:
- board text added: "Bq/m2 uSv/h"
- board text added: "CNT"
- board text added: "GPS FIX"
- board text added: "LED"
- board text added: "LOG"
- board text added: "LOG/ALARM"
- board text added: "OFF"
- board text added: "ON"
- board text added: "POWER"
- board text added: "USER"
- board text added: "iRover"
- board text added: "log cpm"
- board text removed: "BATTERY"
- board text removed: "CHARGING"
- board text removed: "FIX"
- board text removed: "FLASH LOG/ALARM SOUND"
- board text removed: "Institute IRNAS Rače www.irnas.eu"
- board text removed: "Integrated Safecast bGeigie Nano"
- board text removed: "LOG/ ALARM"
- board text removed: "LOG/COUNT"
- board text removed: "OFF/ON"
