File: KiCAD project/kicad_project_geiger.kicad_pcb (KiCad board)
At the start: 2 copper layers, 66.8 x 104.8 mm, 88 parts, among them P1 uFL_conn, P2 I2C_connector, P4 I ROVER, P7 BATTERY, Q1 ZXMP6A13F, Q2 RSR010N10FHATL, Q3 RSR010N10FHATL, Q4 ZXMP6A13F, Q5 BC847C, Q6 RSR010N10FHATL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

Commit message: Update
Parts:
- added G***: LOGO, opensource_hardware:LOGO, B.Cu at (146.5, 85.5)
- added G***: LOGO, opensource_hardware:LOGO, F.Cu at (145.9, 76.3)
- added G***: LOGO, safecast_logo:LABEL, B.Cu at (141.8, 111.5)
- Q7, R21, U14, U15: moved to B.Cu
- R8: moved to F.Cu
- moved U14 55.2 mm to (155.5, 135.2), turned to 90 degrees
- moved U15 44.0 mm to (162.1, 139.9)
- moved Q7 39.1 mm to (162.1, 135.8)
- moved Q1 36.4 mm to (155.5, 138.9), turned to 270 degrees
- moved R21 32.8 mm to (165.6, 138.1), turned to 270 degrees
- moved R8 29.4 mm to (161.1, 131.6), turned to 270 degrees
- moved D6 29.3 mm to (165.8, 153.6)
Routing:
- net +3V3: track 211.7 -> 415.6 mm, vias 6 -> 11
- net GND: track 461.4 -> 656.3 mm, vias 11 -> 29
- net VBAT: track 5.81 -> 118.8 mm, vias 1 -> 5
- net PWR_ON: track 61.5 -> 167.5 mm, vias 1 -> 3
- net I2C_SDA: track 49.6 -> 143.6 mm, vias 0 -> 4
- net I2C_SCL: track 50.1 -> 137.8 mm, vias 1 -> 3
- net PWR: track 5.76 -> 89.7 mm, vias 0 -> 2
- net ENC_B: track 0.00 -> 82.0 mm, vias 0 -> 2
- net ENC_A: track 0.00 -> 78.3 mm, vias 0 -> 4
- net LCD_RST: track 60.3 -> 127.1 mm, vias 1 -> 2
- net ENC_SW: track 29.0 -> 91.2 mm, vias 1 -> 3
- net PWR_OFF: track 3.65 -> 65.1 mm, vias 0 -> 2
- net IROVER: track 82.6 -> 138.7 mm, vias 0 -> 2
- net CS_LOG: track 21.8 -> 77.0 mm, vias 0 -> 2
- net SPI_SCK: track 18.2 -> 72.7 mm, vias 0 -> 2
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- added copper zone on B.Cu, net GND
- added copper zone on F.Cu, net GND
Other:
- board text added: "Institute IRNAS Rače www.irnas.eu"
- board text added: "Integrated Safecast bGeigie"

Commit message: Update
Parts:
- added C19: 10uF, RedBear:TantalC_SizeB_EIA-3528_HandSoldering, B.Cu at (171.2, 137.7)
- moved C7 10.3 mm to (154.6, 106.2), turned to 180 degrees
- moved R6 10.3 mm to (144.3, 103.6), turned to 180 degrees
- moved R7 10.3 mm to (144.3, 106.4), turned to 180 degrees
- moved C6 10.2 mm to (154.6, 103.6), turned to 180 degrees
- moved C10 0.15 mm to (149.4, 109.9), turned to 0 degrees
Connections:
- U10 pad 1: VBAT -> LDO
Routing:
- net VBAT: track 118.8 -> 99.9 mm, vias 5 -> 4
- net LDO: track 50.7 -> 67.7 mm, vias 2 -> 3
- net +3V3: track 415.6 -> 405.2 mm, vias 11 -> 10
- net I2C_SDA: track 143.6 -> 137.3 mm
- net I2C_SCL: track 137.8 -> 133.7 mm
- net PWR: track 89.7 -> 92.6 mm
- net GND: track 656.3 -> 658.9 mm
- net VDD_A: track 19.8 -> 21.4 mm
Other:
- board text added: "GPS"

Commit message: Update
Parts:
- added C20: 1uF, RedBear:R_0603_HandSoldering, F.Cu at (134.5, 93.6)
- turned C3 to 0 degrees
- turned L1 to 0 degrees
Connections:
- C3 pad 1: GND -> Net-(C20-Pad1)
- C3 pad 2: Net-(C3-Pad2) -> GND
- L1 pad 1: +3V3 -> Net-(C20-Pad1)
- L1 pad 2: Net-(C3-Pad2) -> +3V3
- U1 pad 1: Net-(C3-Pad2) -> Net-(C20-Pad1)
Routing:
- net Net-(C20-Pad1): track 0.00 -> 7.94 mm
- net Net-(C3-Pad2): track 5.84 -> 0.00 mm
- net GND: track 658.9 -> 660.0 mm, vias 29 -> 31
