File: KiCAD project/kicad_project_geiger.sch (KiCad schematic (older format))
At the start: 61 parts, among them P4 I ROVER, P7 BATTERY, Q1 2SC1815, Q2 2SC1815, SW1 SWITCH_INV, SW2 SW_DIP_3, SW4 2MD3T2B2M2RE, U1 FGPMMOPA6H, U10 MIC5205, U11 piezo_buzzer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

Commit message: Update
Parts:
- U1: Field4 (none) -> GPS
- U12: Field4 (none) -> Audio Out
- U8: Field4 (none) -> Accelerometer & Magnetometer
Other:
- note added: "RED BEAR"
- moved on the sheet: C16, C17, C8, P4, R15, R16, R8, SW4, U5

Commit message: Update
Parts:
- removed C16: 100nF, RedBear:R_0603_HandSoldering, symbol C
- removed D6: 1N4148, RedBear:1N4148, symbol D
- removed Q1, Q2: 2SC1815, 2SC1815:TO-92_Inline_Narrow_Oval, symbol 2SC1815
- removed SW4: 2MD3T2B2M2RE, TSM102C3_toggle_switch_tme:TSM102C3_toggle_switch, symbol SWITCH_INV
- removed U12: stereo_audio_socket, CLIFF_ELECTRONIC_COMPONENTS_FC68131_PhoneAudioConnector:CLIFF_ELECTRONIC_COMPONENTS_FC68131_PhoneAudioConnector, symbol stereo_audio_socket
- added D6: BAT20J, symbol BAT20J
- added Q1, Q4: ZXMP6A13F, SOT23, symbol ZXMP6A13F
- added Q2, Q3, Q6, Q7: RSR010N10FHATL, SOT-23, symbol RSR010N10FHATL
- added Q5: BC847C, symbol BC847C
- added R20: 68R, RedBear:R_0603_HandSoldering, symbol R
- added R21, R22, R23: 10K, RedBear:R_0603_HandSoldering, symbol R
- added R24, R25: 0K, RedBear:R_0603_HandSoldering, symbol R
- added SW3: SWITCH_INV, OS102011MA1QN1_slide_switch:OS102011MA1QN1_slide_switch, symbol SWITCH_INV
- added SW4: SW_PUSH, KSEK43J_LFS_TACTILE_SWITCH:KSEK43J_LFS_TACTILE_SWITCH, symbol SW_PUSH
- added U12: uFL_conn, symbol uFL_conn
- D2: Field5 (none) -> KPD-3224SURCK
- D3: value BLUE -> GREEN; Field5 (none) -> MCL053SGC
- R12: value 1K -> 10K
- R14: value 100K -> 51K
- R15: value 47K -> 10K
- R16: value 4.7K -> 10K
- R19: value 180K -> 10K
- R8: value 10K -> 100K
- SW1: Function (none) -> POWER
- U11: value piezo_buzzer -> buzzer; footprint CEM-1203(42)_piezo_buzzer:CEM-1203(42) -> (none); Field4 (none) -> LD-BZEG-1205
Connections:
- net labels added: ANALOG, BAT_MEASURE, CNT_LED, LDO, LOG_LED, PIEZO, PWR, PWR_OFF, PWR_ON
- net labels removed: LCD_CS, LCD_DC, LOG_ALARM, LOG_CNT_SEL
- wire segments 99 -> 125
- no-connect marks 41 -> 40
Other:
- note removed: "POWER"
- moved on the sheet: C1, C10, C11, C13, C14, C15, C17, C2, C3, C4, C5, C6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

Commit message: Update
Parts:
- added L1: Ferrite, RedBear:R_0603_HandSoldering, symbol INDUCTOR_SMALL
- D2: footprint RedBear:LED_0603_HandSoldering -> KPD-3224SURCK:KPD-3224SURCK
- D3: footprint LEDs:LED-5MM -> MCL053SGC:MCL053SGC
- D4: footprint RedBear:1N4148 -> SOD-323_standard:SOD-323
- D6: footprint (none) -> SOD-323_standard:SOD-323
- P1: renamed from U12; footprint (none) -> UFL-R-SMT:U.FL-R-SMT
- P4: footprint Socket_Strips:Socket_Strip_Angled_1x03 -> B3B-PH-SM4-TB_IROVER_CONNECTOR:B3B-PH-SM4-TB_IROVER_CONNECTOR
- Q1, Q4: footprint SOT23 -> sot_32_standard:SOT-23
- Q2, Q3, Q6, Q7: footprint SOT-23 -> sot_32_standard:SOT-23
- Q5: footprint (none) -> sot_32_standard:SOT-23
- SW2: Field4 (none) -> A6S-3102-H
- U11: footprint (none) -> LD-BZEG-1205:LD-BZEG-1205
Connections:
- net +3V3: now also L1.1; no longer C3.2, U1.1 (VCC)
- net IROVER: no longer Q2.1 (G), R12.2
- net AUDIO: now reaches U7.19 (D14/A6/UART2_RTS/PA1)
- net AUDIO: now also Q2.1 (G), R12.2
- net at U1.5 (3D_FIX): now also R18.1; no longer R18.2
- net at D5.2 (A): now also R18.2; no longer R18.1
- new net: C3.2, L1.2, U1.1 (VCC)
- no-connect marks 40 -> 39
Other:
- moved on the sheet: D5, R18
