File: KiCAD project/kicad_project_geiger.sch (KiCad schematic (older format))
At the start: 72 parts, among them P4 I ROVER, P7 BATTERY, Q1 ZXMP6A13F, Q2 RSR010N10FHATL, Q3 RSR010N10FHATL, Q4 ZXMP6A13F, Q5 BC847C, Q6 RSR010N10FHATL, Q7 RSR010N10FHATL, SW1 SWITCH_INV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

Commit message: Update
Parts:
- removed Q7: RSR010N10FHATL, SOT-23, symbol RSR010N10FHATL
- removed R21, R22, R23: 10K, RedBear:R_0603_HandSoldering, symbol R
- removed SW3: SWITCH_INV, OS102011MA1QN1_slide_switch:OS102011MA1QN1_slide_switch, symbol SWITCH_INV
- removed SW4: SW_PUSH, KSEK43J_LFS_TACTILE_SWITCH:KSEK43J_LFS_TACTILE_SWITCH, symbol SW_PUSH
- added C16, C18: 10nF, RedBear:R_0603_HandSoldering, symbol C
- added L1: Ferrite, RedBear:R_0603_HandSoldering, symbol INDUCTOR_SMALL
- added P2: I2C_connector, DIP Grove 4P-2.0:DIP_Grove_4P-2_0, symbol I2C_connector
- added R26: 0R, RedBear:R_0603_HandSoldering, symbol R
- added R27, R28, R29, R30, R31, R32, R33: 10K, RedBear:R_0603_HandSoldering, symbol R
- added U12: rotary_encoder, rotary_enc_bourns_EC12R-4215F-S0024:rotary_enc_bourns_EC12R-4215F-S0024, symbol rotary_encoder
- D2: footprint RedBear:LED_0603_HandSoldering -> KPD-3224SURCK:KPD-3224SURCK
- D3: footprint LEDs:LED-5MM -> MCL053SGC:MCL053SGC
- D4: footprint RedBear:1N4148 -> SOD-323_standard:SOD-323
- D6: footprint (none) -> SOD-323_standard:SOD-323
- P1: renamed from U12; footprint (none) -> UFL-R-SMT:U.FL-R-SMT
- P4: footprint Socket_Strips:Socket_Strip_Angled_1x03 -> B3B-PH-SM4-TB_IROVER_CONNECTOR:B3B-PH-SM4-TB_IROVER_CONNECTOR
- Q1, Q4: footprint SOT23 -> sot_32_standard:SOT-23
- Q2, Q3, Q6: footprint SOT-23 -> sot_32_standard:SOT-23
- Q5: footprint (none) -> sot_32_standard:SOT-23
- SW2: Field4 (none) -> A6S-3102-H
- U11: footprint (none) -> LD-BZEG-1205:LD-BZEG-1205
Connections:
- net labels added: ENC_A, ENC_B, ENC_SW
- net labels removed: ANALOG
- wire segments 125 -> 141
- no-connect marks 40 -> 37
Other:
- moved on the sheet: C4, D5, R18, R19, U7
